Commit message: initial commit & xacro params.yaml changed

File: launch/include/config/robot.urdf.xacro (robot description, xacro)
@@ -2,14 +2,20 @@
 <robot name="roboat" xmlns:xacro="http://roboat.org">
   <xacro:property name="PI" value="3.1415926535897931" />
+  <link name="odom"></link>
   <link name="base_link"></link>
+  <link name="base_link_gt"></link>
   <joint name="base_link_joint" type="fixed">
-    <parent link="base_link"/>
-    <child link="chassis_link" />
+    <parent link="odom"/>
+    <child link="base_link" />
     <origin xyz="0 0 0" rpy="0 0 0" />
   </joint>
-  <link name="chassis_link"></link>
+  <joint name="odom_joint" type="fixed">
+  <parent link="odom"/>
+  <child link="base_link_gt" />
+  <origin xyz="0 0 0" rpy="0 0 0" />
+  </joint>
   <link name="imu_link"> </link>
   <joint name="imu_joint" type="fixed">
-    <parent link="chassis_link" />
+    <parent link="base_link_gt" />
     <child link="imu_link" />
     <origin xyz="0 -0.1 0" rpy="${PI} 0 ${PI}" />
@@ -23,5 +29,5 @@
   <link name="velodyne"> </link>
   <joint name="velodyne_joint" type="fixed">
-    <parent link="chassis_link" />
+    <parent link="base_link_gt" />
     <child link="velodyne" />
     <origin xyz="0 0 0" rpy="0 0 0" />
@@ -29,5 +35,5 @@
   <link name="realsense_link"> </link>
   <joint name="realsense_joint" type="fixed">
-    <parent link="chassis_link" />
+    <parent link="base_link_gt" />
     <child link="realsense_link" />
     <origin xyz="0.1 0 -0.1" rpy="0 0 0" />
@@ -35,5 +41,5 @@
   <link name="navsat_link"> </link>
   <joint name="navsat_joint" type="fixed">
-    <parent link="chassis_link" />
+    <parent link="base_link_gt" />
     <child link="navsat_link" />
     <origin xyz="-0.2 0 0.2" rpy="0 0 0" />
@@ -41,5 +47,5 @@
   <link name="loam_camera"> </link>
   <joint name="_loam_camera_joint" type="fixed">
-    <parent link="chassis_link" />
+    <parent link="base_link_gt" />
     <child link="loam_camera" />
     <origin xyz="0 0 0" rpy="1.570796 0 1.570796" />
